File: tbthanh-try-ai03-pcb-guide.sch (KiCad schematic (older format))
At the start: 24 parts, among them SW1 SW_Push, U1 ATmega32U4-AU, Y1 16MHz

Commit message: 1st pcb done but too tired.
Good night
Connections:
- net +5V: now also U1.24 (AVCC), U1.44 (AVCC)
- net COL0: now also U1.29 (PB5)
- net COL1: now also U1.28 (PB4)
- net GND: now also U1.15 (GND), U1.23 (GND), U1.35 (GND), U1.43 (GND)
- net ROW0: now also U1.27 (PD7)
- net ROW1: now also U1.30 (PB6)
Changed lines of the file:
@@
 	3850 1350 3850 1700
 Connection ~ 3850 1700
+Text GLabel 4550 3900 2    50   Input ~ 0
+ROW0
+Text GLabel 4550 2600 2    50   Input ~ 0
+ROW1
+Text GLabel 4550 2500 2    50   Input ~ 0
+COL0
+Text GLabel 4550 2400 2    50   Input ~ 0
+COL1
+Wire Wire Line
+	3950 5300 3850 5300
+Connection ~ 3850 5300
+Wire Wire Line
+	3950 1700 4050 1700
+Connection ~ 3950 1700
 $EndSCHEMATC
